Commit message: Changed range for left arm joints

File: tesseract_py/resource/g1.urdf (robot description, URDF)
Before this commit: robot g1, 73 links, 72 joints
Joints:
- joint left_elbow_joint: limit lower=-1.0472 upper=2.0944 effort=25 velocity=37.0 -> lower=-0.9 upper=2.0 effort=25 velocity=37.0
- joint left_shoulder_pitch_joint: limit lower=-3.0892 upper=2.6704 effort=25 velocity=37.0 -> lower=-2.9 upper=2.5 effort=25 velocity=37.0
- joint left_shoulder_roll_joint: limit lower=-1.5882 upper=2.2515 effort=25 velocity=37.0 -> lower=-1.4 upper=2.1 effort=25 velocity=37.0
- joint left_shoulder_yaw_joint: limit lower=-2.618 upper=2.618 effort=25 velocity=37.0 -> lower=-2.5 upper=2.5 effort=25 velocity=37.0
- joint left_wrist_roll_joint: limit lower=-1.972222054 upper=1.972222054 effort=25 velocity=37.0 -> lower=-1.8 upper=1.8 effort=25 velocity=37.0
